Commit message: Added collision and inertial

File: description/gripper_fingers.xacro (robot description, xacro)
@@ -1,9 +1,10 @@
 <?xml version="1.0"?>
-<robot xmlns:xacro="http://www.ros.org/wiki/xacro"  name="robot">
+<robot xmlns:xacro="http://www.ros.org/wiki/xacro"  >
+    <xacro:include filename="inertial_macros.xacro" />
     <xacro:macro name="finger" params="id yaw">
                             <!-- FINGER-->
     <!-- BOTTOM-->
     <joint name="${id}_finger_bottom_joint" type="revolute" >
-        <limit effort="5" velocity="2.1750" lower="-0.5" upper="0.5"/>
+        <limit effort="5" velocity="2.1750" lower="-0.1" upper="0.5"/>
         <parent link="last_arm_link" />
         <child link="${id}_finger_bottom_link" />
@@ -19,4 +20,13 @@
             <material name="black"/>
         </visual>
+        <collision>
+            <origin xyz="0 0 0.15" rpy="0 0 0 "/>
+            <geometry>
+                <box size="0.025 0.025 0.3"/>
+            </geometry>
+        </collision>
+        <xacro:inertial_box mass="0.05" x="0.025" y="0.025" z="0.3" >
+            <origin xyz="0 0 0.15" rpy="0 0 0" />
+        </xacro:inertial_box>
     </link>
     <!-- TOP-->
@@ -34,4 +44,13 @@
             <material name="white"/>
         </visual>
+        <collision>
+            <origin xyz="0 0 0.15" rpy="0 0 0 "/>
+            <geometry>
+                <box size="0.025 0.025 0.3"/>
+            </geometry>
+        </collision>
+        <xacro:inertial_box mass="0.05" x="0.025" y="0.025" z="0.3" >
+            <origin xyz="0 0 0.15" rpy="0 0 0" />
+        </xacro:inertial_box>
     </link>
     </xacro:macro>
