Commit message: Gripper fingers maded with macros.Robot skeleton is builded

File: description/robot_core.xacro (robot description, xacro)
@@ -1,4 +1,7 @@
 <?xml version="1.0"?>
 <robot xmlns:xacro="http://www.ros.org/wiki/xacro"  >
+    <material name="black">
+        <color rgba="0 0 0 1"/>
+    </material>
     <material name="white">
         <color rgba="1 1 1 1"/>
@@ -6,17 +9,137 @@
     <link name="base_link">
     </link>
-    <joint name="chassis_joint" type="fixed">
+       <!-- CHASSIS -->
+    <joint name="chassis_joint" type="revolute">
+        <limit effort="5" velocity="2.1750" lower="-3.14" upper="3.14"/>
         <parent link="base_link"/>
-        <child link="chassis" />
+        <child link="chassis_link" />
         <origin xyz="0 0 0"/>
+        <axis xyz="0 0 1" />
     </joint>
-    <link name="chassis">
+    <link name="chassis_link">
         <visual>
-            <origin xyz="0.4 0.4 0.4"/>
+            <origin xyz="0 0 0.2"/>
             <geometry>
-                <box size="0.8 0.8 0.8" />
+                <box size="0.8 0.8 0.4" />
             </geometry>
             <material name="white"/>
         </visual>
     </link>
+       <!-- BASE LOWER ARM -->
+    <joint name="base_lower_arm_joint" type="fixed">
+        <parent link="chassis_link" />
+        <child link="base_lower_arm_link" />
+        <origin xyz="0 0 0.4" />
+    </joint>
+    <link name="base_lower_arm_link">
+        <visual>
+            <origin xyz="0 0.02 0.1" rpy="${pi/2} 0 ${pi/2}"/>
+            <geometry>
+                <cylinder radius="0.2" length="0.8" />
+            </geometry>
+            <material name="white"/>
+        </visual>
+    </link>
+       <!-- LOWER ARM -->
+    <joint name="lower_arm_joint" type="revolute" >
+        <limit effort="5" velocity="2.1750" lower="0" upper="1"/>
+        <parent link="base_lower_arm_link" />
+        <child link="lower_arm_link" />
+        <origin xyz="0 0 0.2" />
+    </joint>
+    <link name="lower_arm_link">
+        <visual>
+            <origin xyz="0 0 0.4"/>
+            <geometry>
+                <box size="0.4 0.4 0.8"/>
+            </geometry>
+            <material name="white"/>
+        </visual>
+    </link>
+       <!-- BASE UPPER ARM -->
+    <joint name="base_upper_arm_joint" type="fixed" >
+        <parent link="lower_arm_link" />
+        <child link="base_upper_arm_link" />
+        <origin xyz="0 0 0.8" />
+    </joint>
+    <link name="base_upper_arm_link" >
+        <visual>
+            <origin xyz="0 0 0.05" rpy="${pi/2} 0 ${pi/2}"/>
+            <geometry>
+                <cylinder radius="0.1" length="0.4" />
+            </geometry>
+            <material name="white"/>
+        </visual>
+    </link>
+       <!-- UPPER ARM -->
+    <joint name="upper_arm_joint" type="revolute" >
+        <limit effort="5" velocity="2.1750" lower="0" upper="1"/>
+        <parent link="base_upper_arm_link" />
+        <child link="upper_arm_link" />
+        <origin xyz="0 0 0.1" />
+    </joint>
+    <link name="upper_arm_link">
+        <visual>
+            <origin xyz="0 0 0.4"/>
+            <geometry>
+                <box size="0.4 0.4 0.8"/>
+            </geometry>
+            <material name="white"/>
+        </visual>
+    </link>
+       <!-- YAW ARM  -->
+    <joint name="yaw_arm_joint" type="revolute" >
+        <limit effort="5" velocity="2.1750" lower="-3.14" upper="3.14"/>
+        <parent link="upper_arm_link" />
+        <child link="yaw_arm_link" />
+        <origin xyz="0 0 0.8" />
+        <axis xyz="0 0 1" />
+    </joint>
+    <link name="yaw_arm_link">
+        <visual>
+            <origin xyz="0 0 0.005"/>
+            <geometry>
+                <cylinder radius="0.2" length="0.01"/>
+            </geometry>
+            <material name="white"/>
+        </visual>
+    </link>
+       <!-- BASE CYLINDER LAST ARM -->
+    <joint name="base_last_arm_joint" type="fixed" >
+        <parent link="yaw_arm_link" />
+        <child link="base_last_arm_link" />
+        <origin xyz="0 0 0.01" />
+    </joint>
+    <link name="base_last_arm_link" >
+        <visual>
+            <origin xyz="0 0 0.05" rpy="${pi/2} 0 ${pi/2}"/>
+            <geometry>
+                <cylinder radius="0.1" length="0.4" />
+            </geometry>
+            <material name="white"/>
+        </visual>
+    </link>
+       <!-- LAST ARM -->
+    <joint name="last_arm_joint" type="revolute" >
+        <limit effort="5" velocity="2.1750" lower="-1" upper="1"/>
+        <parent link="base_last_arm_link" />
+        <child link="last_arm_link" />
+        <origin xyz="0 0 0.1" />
+    </joint>
+    <link name="last_arm_link">
+        <visual>
+            <origin xyz="0 0 0.15"/>
+            <geometry>
+                <box size="0.15 0.15 0.3"/>
+            </geometry>
+            <material name="white"/>
+        </visual>
+    </link>
+    <!-- GRIPPER -->
+    <!-- FINGERS MACRO -->
+    <xacro:include filename="gripper_fingers.xacro" />
+    <xacro:finger id="first" yaw="${pi/4}"/>
+    <xacro:finger id="second" yaw="${3*pi/4}"/>
+    <xacro:finger id="third" yaw="${5*pi/4}"/>
+    <xacro:finger id="fourth" yaw="${7*pi/4}"/>
 </robot>

File: description/templates.xacro (robot description, xacro)
@@ -7,4 +7,5 @@
                 <box size="0.3 0.3 0.15" />
             </geometry>
+        </visual>
     </link>
     <!-- Example material -->

Commit message: Created macros,added inertial and collision

File: description/robot_core.xacro (robot description, xacro)
@@ -1,4 +1,6 @@
 <?xml version="1.0"?>
 <robot xmlns:xacro="http://www.ros.org/wiki/xacro"  >
+    <xacro:include filename="joint_macro.xacro" />
+    <xacro:include filename="gripper_fingers.xacro" />
     <material name="black">
         <color rgba="0 0 0 1"/>
@@ -26,67 +28,17 @@
         </visual>
     </link>
-       <!-- BASE LOWER ARM -->
-    <joint name="base_lower_arm_joint" type="fixed">
-        <parent link="chassis_link" />
-        <child link="base_lower_arm_link" />
-        <origin xyz="0 0 0.4" />
-    </joint>
-    <link name="base_lower_arm_link">
-        <visual>
-            <origin xyz="0 0.02 0.1" rpy="${pi/2} 0 ${pi/2}"/>
-            <geometry>
-                <cylinder radius="0.2" length="0.8" />
-            </geometry>
-            <material name="white"/>
-        </visual>
-    </link>
-       <!-- LOWER ARM -->
-    <joint name="lower_arm_joint" type="revolute" >
-        <limit effort="5" velocity="2.1750" lower="0" upper="1"/>
-        <parent link="base_lower_arm_link" />
-        <child link="lower_arm_link" />
-        <origin xyz="0 0 0.2" />
-    </joint>
-    <link name="lower_arm_link">
-        <visual>
-            <origin xyz="0 0 0.4"/>
-            <geometry>
-                <box size="0.4 0.4 0.8"/>
-            </geometry>
-            <material name="white"/>
-        </visual>
-    </link>
-       <!-- BASE UPPER ARM -->
-    <joint name="base_upper_arm_joint" type="fixed" >
-        <parent link="lower_arm_link" />
-        <child link="base_upper_arm_link" />
-        <origin xyz="0 0 0.8" />
-    </joint>
-    <link name="base_upper_arm_link" >
-        <visual>
-            <origin xyz="0 0 0.05" rpy="${pi/2} 0 ${pi/2}"/>
-            <geometry>
-                <cylinder radius="0.1" length="0.4" />
-            </geometry>
-            <material name="white"/>
-        </visual>
-    </link>
-       <!-- UPPER ARM -->
-    <joint name="upper_arm_joint" type="revolute" >
-        <limit effort="5" velocity="2.1750" lower="0" upper="1"/>
-        <parent link="base_upper_arm_link" />
-        <child link="upper_arm_link" />
-        <origin xyz="0 0 0.1" />
-    </joint>
-    <link name="upper_arm_link">
-        <visual>
-            <origin xyz="0 0 0.4"/>
-            <geometry>
-                <box size="0.4 0.4 0.8"/>
-            </geometry>
-            <material name="white"/>
-        </visual>
-    </link>
-       <!-- YAW ARM  -->
+    <!-- BASE LOWER ARM -->
+    <xacro:base_arm_generator suffix="lower" parent="chassis" ph="0.4" radius="0.2" length="0.8" />
+    <!-- BASE UPPER ARM -->
+    <xacro:base_arm_generator suffix="upper" parent="lower_arm" ph="0.8" radius="0.1" length="0.4" />
+    <!-- BASE LAST ARM -->
+    <xacro:base_arm_generator suffix="last" parent="yaw_arm" ph="0.01" radius="0.1" length="0.4" />
+    <!-- LOWER ARM -->
+    <xacro:arm_generator suffix="lower" parent="base_lower_arm" ph="0.2" sizex="0.4"  sizey="0.4" sizez="0.8" upper="1" lower="0" />
+    <!-- UPPER ARM -->
+    <xacro:arm_generator suffix="upper" parent="base_upper_arm" ph="0.1" sizex="0.4"  sizey="0.4" sizez="0.8" upper="1" lower="0" />
+    <!-- LAST ARM -->
+    <xacro:arm_generator suffix="last"  parent="base_last_arm"  ph="0.1" sizex="0.15" sizey="0.15" sizez="0.3" upper="1" lower="-1" />
+    <!-- YAW ARM  -->
     <joint name="yaw_arm_joint" type="revolute" >
         <limit effort="5" velocity="2.1750" lower="-3.14" upper="3.14"/>
@@ -105,38 +57,6 @@
         </visual>
     </link>
-       <!-- BASE CYLINDER LAST ARM -->
-    <joint name="base_last_arm_joint" type="fixed" >
-        <parent link="yaw_arm_link" />
-        <child link="base_last_arm_link" />
-        <origin xyz="0 0 0.01" />
-    </joint>
-    <link name="base_last_arm_link" >
-        <visual>
-            <origin xyz="0 0 0.05" rpy="${pi/2} 0 ${pi/2}"/>
-            <geometry>
-                <cylinder radius="0.1" length="0.4" />
-            </geometry>
-            <material name="white"/>
-        </visual>
-    </link>
-       <!-- LAST ARM -->
-    <joint name="last_arm_joint" type="revolute" >
-        <limit effort="5" velocity="2.1750" lower="-1" upper="1"/>
-        <parent link="base_last_arm_link" />
-        <child link="last_arm_link" />
-        <origin xyz="0 0 0.1" />
-    </joint>
-    <link name="last_arm_link">
-        <visual>
-            <origin xyz="0 0 0.15"/>
-            <geometry>
-                <box size="0.15 0.15 0.3"/>
-            </geometry>
-            <material name="white"/>
-        </visual>
-    </link>
     <!-- GRIPPER -->
     <!-- FINGERS MACRO -->
-    <xacro:include filename="gripper_fingers.xacro" />
     <xacro:finger id="first" yaw="${pi/4}"/>
     <xacro:finger id="second" yaw="${3*pi/4}"/>
